Commit message: Update urdf

File: lz01/LZ01_Lite_V3.urdf (robot description, URDF)
Before this commit: robot LZ01_Lite_V3, 27 links, 26 joints
Links:
- added link left_hand_tip
- added link right_hand_tip
Joints:
- added joint left_elbow_to_hand_tip: type fixed, parent left_elbow_link, child left_hand_tip, origin xyz=0 0 -0.24 rpy=0 0 0
- added joint right_elbow_to_hand_tip: type fixed, parent right_elbow_link, child right_hand_tip, origin xyz=0 0 -0.24 rpy=0 0 0
- joint torso_yaw_link_to_camera_link: origin xyz=0.01 0 0.3225 rpy=0 0.651 0 -> xyz=0.0441828 0 0.32325 rpy=0 0.349066 0
